File: MCU.sch (KiCad schematic (older format))
At the start: 11 parts, among them J4 Conn_01x02, J5 AVR-ISP-6, SW2 SW_SPDT, U4 ATTINY13

Commit message: Preparing for v1.2 Updated to KiCAD 5 nightly Added resistors to isolate the programming pins Added transistor to drive the LED Replaced LTC3458 boost converter with an LTC3536 buck-boost converter to step down the USB power supply Added debugging jumper to test the voltage regulator
Parts:
- added Q3: MMBT3904, TO_SOT_Packages_SMD:SOT-23, symbol transistors:MMBT3904
- added R17, R18: 4.7k, Resistors_SMD:R_0603, symbol device:R
- C10: renamed from C12; symbol C -> device:C
- C11: renamed from C13; symbol C -> device:C
- C12: renamed from C14; symbol C -> device:C
- J6: renamed from J4; symbol Conn_01x02 -> conn:Conn_01x02
- J7: renamed from J5; symbol AVR-ISP-6 -> atmel:AVR-ISP-6
- R13: renamed from R14; symbol R -> device:R
- R14: renamed from R15; symbol R -> device:R
- R15: renamed from R16; symbol R -> device:R
- R16: renamed from R17; symbol R -> device:R
- SW2: symbol SW_SPDT -> switches:SW_SPDT
- U4: symbol ATTINY13-20SSU -> atmel:ATTINY13-20SSU
Connections:
- net GND: now also Q3.2 (E); no longer J6.2 (Pin_2)
- net MISO: now also R18.2; no longer R15.1
- net Vdd: now also R15.1
- net kill_power renamed MOSI
- net MOSI: now also R17.2
- new net: J6.2 (Pin_2), Q3.3 (C)
- new net: Q3.1 (B), R18.1
- new net ~kill_power: R17.1
Other:
- note added: "We are using a transistor\nso that we can isolate the\npin using a 4.7k resistor"
- moved on the sheet: J6, R15
Changed lines of the file:
@@
-EESchema Schematic File Version 2
-LIBS:power
-LIBS:device
-LIBS:transistors
-LIBS:conn
-LIBS:linear
-LIBS:regul
-LIBS:74xx
-LIBS:cmos4000
-LIBS:adc-dac
-LIBS:memory
-LIBS:xilinx
-LIBS:microcontrollers
-LIBS:dsp
-LIBS:microchip
-LIBS:analog_switches
-LIBS:motorola
-LIBS:texas
-LIBS:intel
-LIBS:audio
-LIBS:interface
-LIBS:digital-audio
-LIBS:philips
-LIBS:display
-LIBS:cypress
-LIBS:siliconi
-LIBS:opto
-LIBS:atmel
-LIBS:contrib
-LIBS:valves
-LIBS:switches
-LIBS:Microchip
-LIBS:On Semiconductor
-LIBS:Linear Technology
+EESchema Schematic File Version 4
 LIBS:main-cache
 EELAYER 26 0
@@
 ~enable_heater
 $Comp
-L R R14
+L device:R R13
 U 1 1 59D0B837
 P 5550 4550
-F 0 "R14" V 5343 4550 50  0000 C CNN
+F 0 "R13" V 5343 4550 50  0000 C CNN
 F 1 "1k" V 5434 4550 50  0000 C CNN
 F 2 "Resistors_SMD:R_0603" V 5480 4550 50  0001 C CNN
@@
 $EndComp
 $Comp
-L C C13
+L device:C C11
 U 1 1 59D0B89F
 P 5850 4800
-F 0 "C13" H 5965 4846 50  0000 L CNN
+F 0 "C11" H 5965 4846 50  0000 L CNN
 F 1 "100n" H 5965 4755 50  0000 L CNN
 F 2 "Capacitors_SMD:C_0603" H 5888 4650 50  0001 C CNN
@@
 $EndComp
 $Comp
-L GND #PWR028
+L power:GND #PWR026
 U 1 1 59D0B8EA
 P 5850 5050
-F 0 "#PWR028" H 5850 4800 50  0001 C CNN
+F 0 "#PWR026" H 5850 4800 50  0001 C CNN
 F 1 "GND" H 5855 4877 50  0000 C CNN
 F 2 "" H 5850 5050 50  0001 C CNN
@@
 $EndComp
 $Comp
-L ATTINY13-20SSU U4
+L atmel:ATTINY13-20SSU U4
 U 1 1 59D0BE2F
 P 5300 3250
@@
 $EndComp
 $Comp
-L GND #PWR029
+L power:GND #PWR025
 U 1 1 59D0C06D
 P 4100 3600
-F 0 "#PWR029" H 4100 3350 50  0001 C CNN
+F 0 "#PWR025" H 4100 3350 50  0001 C CNN
 F 1 "GND" H 4105 3427 50  0000 C CNN
 F 2 "" H 4100 3600 50  0001 C CNN
@@
 $EndComp
 $Comp
-L GND #PWR030
+L power:GND #PWR030
 U 1 1 59D0C22E
 P 8000 2750
@@
 Vdd
 $Comp
-L R R17
+L device:R R16
 U 1 1 59D0C448
 P 8600 2900
-F 0 "R17" H 8670 2946 50  0000 L CNN
+F 0 "R16" H 8670 2946 50  0000 L CNN
 F 1 "10k" H 8670 2855 50  0000 L CNN
 F 2 "Resistors_SMD:R_0603" V 8530 2900 50  0001 C CNN
@@
 $EndComp
 $Comp
-L C C12
+L device:C C10
 U 1 1 59D0C55B
 P 3700 3400
-F 0 "C12" H 3815 3446 50  0000 L CNN
+F 0 "C10" H 3815 3446 50  0000 L CNN
 F 1 "100n" H 3815 3355 50  0000 L CNN
 F 2 "Capacitors_SMD:C_0603" H 3738 3250 50  0001 C CNN
@@
 $EndComp
 $Comp
-L GND #PWR031
+L power:GND #PWR024
 U 1 1 59D0C561
 P 3700 3650
-F 0 "#PWR031" H 3700 3400 50  0001 C CNN
+F 0 "#PWR024" H 3700 3400 50  0001 C CNN
 F 1 "GND" H 3705 3477 50  0000 C CNN
 F 2 "" H 3700 3650 50  0001 C CNN
@@
 	1    0    0    -1
 $EndComp
-Text HLabel 7650 4050 2    60   Output ~ 0
-kill_power
-$Comp
-L R R16
+Text HLabel 8200 4050 2    60   Output ~ 0
+~kill_power
+$Comp
+L device:R R15
 U 1 1 59D0EA56
-P 7150 4350
-F 0 "R16" H 7220 4396 50  0000 L CNN
-F 1 "470" H 7220 4305 50  0000 L CNN
-F 2 "Resistors_SMD:R_0603" V 7080 4350 50  0001 C CNN
-F 3 "" H 7150 4350 50  0001 C CNN
-F 4 "Yageo" H 7150 4350 60  0001 C CNN "MFN"
-F 5 "RC0603FR-07470RL" H 7150 4350 60  0001 C CNN "MFP"
-	1    7150 4350
-	1    0    0    -1
-$EndComp
-$Comp
-L GND #PWR032
+P 8650 4850
+F 0 "R15" H 8720 4896 50  0000 L CNN
+F 1 "470" H 8720 4805 50  0000 L CNN
+F 2 "Resistors_SMD:R_0603" V 8580 4850 50  0001 C CNN
+F 3 "" H 8650 4850 50  0001 C CNN
+F 4 "Yageo" H 8650 4850 60  0001 C CNN "MFN"
+F 5 "RC0603FR-07470RL" H 8650 4850 60  0001 C CNN "MFP"
+	1    8650 4850
+	1    0    0    -1
+$EndComp
+$Comp
+L power:GND #PWR029
 U 1 1 59D0EBB5
-P 7150 4850
-F 0 "#PWR032" H 7150 4600 50  0001 C CNN
-F 1 "GND" H 7155 4677 50  0000 C CNN
-F 2 "" H 7150 4850 50  0001 C CNN
-F 3 "" H 7150 4850 50  0001 C CNN
-	1    7150 4850
-	1    0    0    -1
-$EndComp
-$Comp
-L SW_SPDT SW2
+P 8650 5850
+F 0 "#PWR029" H 8650 5600 50  0001 C CNN
+F 1 "GND" H 8655 5677 50  0000 C CNN
+F 2 "" H 8650 5850 50  0001 C CNN
+F 3 "" H 8650 5850 50  0001 C CNN
+	1    8650 5850
+	1    0    0    -1
+$EndComp
+$Comp
+L switches:SW_SPDT SW2
 U 1 1 59D116BA
 P 6700 1900
@@
 $EndComp
 $Comp
-L GND #PWR033
+L power:GND #PWR028
 U 1 1 59D11856
 P 7050 1900
-F 0 "#PWR033" H 7050 1650 50  0001 C CNN
+F 0 "#PWR028" H 7050 1650 50  0001 C CNN
 F 1 "GND" H 7055 1727 50  0000 C CNN
 F 2 "" H 7050 1900 50  0001 C CNN
@@
 $EndComp
 $Comp
-L Conn_01x02 J4
+L conn:Conn_01x02 J6
 U 1 1 59D151F1
-P 7400 4650
-F 0 "J4" H 7480 4642 50  0000 L CNN
-F 1 "Conn_01x02" H 7480 4551 50  0000 L CNN
-F 2 "Connectors_JST:JST_PH_B2B-PH-K_02x2.00mm_Straight" H 7400 4650 50  0001 C CNN
-F 3 "" H 7400 4650 50  0001 C CNN
-F 4 "JST" H 7400 4650 60  0001 C CNN "MFN"
-F 5 "B2B-PH-K-S(LF)(SN)" H 7400 4650 60  0001 C CNN "MFP"
-F 6 "Amber LED" H 7400 4650 60  0001 C CNN "Note"
-	1    7400 4650
-	1    0    0    -1
-$EndComp
-$Comp
-L C C14
+P 8900 5150
+F 0 "J6" H 8980 5142 50  0000 L CNN
+F 1 "Conn_01x02" H 8980 5051 50  0000 L CNN
+F 2 "Connectors_JST:JST_PH_B2B-PH-K_02x2.00mm_Straight" H 8900 5150 50  0001 C CNN
+F 3 "" H 8900 5150 50  0001 C CNN
+F 4 "JST" H 8900 5150 60  0001 C CNN "MFN"
+F 5 "B2B-PH-K-S(LF)(SN)" H 8900 5150 60  0001 C CNN "MFP"
+F 6 "Amber LED" H 8900 5150 60  0001 C CNN "Note"
+	1    8900 5150
+	1    0    0    -1
+$EndComp
+$Comp
+L device:C C12
 U 1 1 59D1A6E6
 P 6050 2100
-F 0 "C14" H 6165 2146 50  0000 L CNN
+F 0 "C12" H 6165 2146 50  0000 L CNN
 F 1 "100n" H 6165 2055 50  0000 L CNN
 F 2 "Capacitors_SMD:C_0603" H 6088 1950 50  0001 C CNN
@@
 $EndComp
 $Comp
-L GND #PWR034
+L power:GND #PWR027
 U 1 1 59D1A77F
 P 6050 2300
-F 0 "#PWR034" H 6050 2050 50  0001 C CNN
+F 0 "#PWR027" H 6050 2050 50  0001 C CNN
 F 1 "GND" H 6055 2127 50  0000 C CNN
 F 2 "" H 6050 2300 50  0001 C CNN
@@
 	5250 4550 5400 4550
 Wire Wire Line
-	5700 4550 6550 4550
+	5700 4550 5850 4550
 Wire Wire Line
 	5850 4550 5850 4650
@@
 	5850 4950 5850 5050
 Wire Wire Line
-	3350 3000 4300 3000
+	3350 3000 3700 3000
 Wire Wire Line
 	4300 3500 4100 3500
@@
 	7150 2500 7500 2500
 Wire Wire Line
-	6300 3100 7150 3100
+	6300 3100 6700 3100
 Wire Wire Line
 	7250 2600 7500 2600
@@
 	7250 2600 7250 3200
 Wire Wire Line
-	7250 3200 6300 3200
+	7250 3200 6400 3200
 Wire Wire Line
 	7350 2700 7500 2700
@@
 	7350 2700 7350 3500
 Wire Wire Line
-	6300 3500 8600 3500
-Wire Wire Line
-	6300 3000 8300 3000
+	6300 3500 7350 3500
+Wire Wire Line
+	6300 3000 6850 3000
 Wire Wire Line
 	8300 3000 8300 2600
@@
 Connection ~ 5850 4550
 Wire Wire Line
-	7150 4750 7150 4850
-Wire Wire Line
-	7150 4500 7150 4650
-Wire Wire Line
-	6700 3100 6700 4150
-Wire Wire Line
-	6700 4150 7150 4150
-Wire Wire Line
-	7150 4150 7150 4200
+	8650 5750 8650 5850
+Wire Wire Line
+	8650 5000 8650 5150
 Connection ~ 6700 3100
 Wire Wire Line
-	6050 1900 6500 1900
+	6050 1900 6400 1900
 Wire Wire Line
 	6900 1800 7050 1800
@@
 Connection ~ 6850 3000
 Wire Wire Line
-	7150 4650 7200 4650
-Wire Wire Line
-	7200 4750 7150 4750
+	8650 5150 8700 5150
+Wire Wire Line
+	8700 5250 8650 5250
 Wire Wire Line
 	6050 1900 6050 1950
@@
 	6050 2300 6050 2250
 Wire Wire Line
-	7750 2500 9350 2500
+	7750 2500 8600 2500
 Text Label 6500 3500 0    60   ~ 0
 RST
@@
 	6300 3300 7150 3300
 $Comp
-L R R15
+L device:R R14
 U 1 1 5A46E3DE
 P 6400 2500
-F 0 "R15" H 6470 2546 50  0000 L CNN
+F 0 "R14" H 6470 2546 50  0000 L CNN
 F 1 "4.7k" H 6470 2455 50  0000 L CNN
 F 2 "Resistors_SMD:R_0603" V 6330 2500 50  0001 C CNN
@@
 Connection ~ 6400 3200
 $Comp
-L AVR-ISP-6 J5
+L atmel:AVR-ISP-6 J7
 U 1 1 5A46F178
 P 7650 2600
-F 0 "J5" H 7637 2965 50  0000 C CNN
+F 0 "J7" H 7637 2965 50  0000 C CNN
 F 1 "AVR-ISP-6" H 7637 2874 50  0000 C CNN
 F 2 "Pin_Headers:Pin_Header_Straight_2x03_Pitch2.54mm" V 7130 2640 50  0001 C CNN
@@
 	1    0    0    -1
 $EndComp
+Wire Wire Line
+	8600 2500 9350 2500
+Wire Wire Line
+	7350 3500 8600 3500
+Wire Wire Line
+	3700 3000 4300 3000
+Wire Wire Line
+	5850 4550 6550 4550
+Wire Wire Line
+	6700 3100 7150 3100
+Wire Wire Line
+	6850 3000 8300 3000
+Wire Wire Line
+	6400 1900 6500 1900
+Wire Wire Line
+	6400 3200 6300 3200
+$Comp
+L device:R R17
+U 1 1 5AAF2F34
+P 7800 4050
+F 0 "R17" V 7593 4050 50  0000 C CNN
+F 1 "4.7k" V 7684 4050 50  0000 C CNN
+F 2 "Resistors_SMD:R_0603" V 7730 4050 50  0001 C CNN
+F 3 "" H 7800 4050 50  0001 C CNN
+F 4 "Yageo" H 7800 4050 50  0001 C CNN "MFN"
+F 5 "RC0603FR-074K7L" H 7800 4050 50  0001 C CNN "MFP"
+	1    7800 4050
+	0    1    1    0
+$EndComp
+Wire Wire Line
+	8200 4050 7950 4050
+Text HLabel 8650 4500 1    60   UnSpc ~ 0
+Vdd
+Wire Wire Line
+	8650 4500 8650 4700
+$Comp
+L transistors:MMBT3904 Q3
+U 1 1 5AAF71EA
+P 8550 5550
+F 0 "Q3" H 8741 5596 50  0000 L CNN
+F 1 "MMBT3904" H 8741 5505 50  0000 L CNN
+F 2 "TO_SOT_Packages_SMD:SOT-23" H 8750 5475 50  0001 L CIN
+F 3 "" H 8550 5550 50  0001 L CNN
+F 4 "Nexperia" H 8550 5550 50  0001 C CNN "MFN"
+F 5 "MMBT3904,215" H 8550 5550 50  0001 C CNN "MFP"
+	1    8550 5550
+	1    0    0    -1
+$EndComp
+Wire Wire Line
+	8650 5250 8650 5350
+$Comp
+L device:R R18
+U 1 1 5AAF9A93
+P 8050 5550
+F 0 "R18" V 7843 5550 50  0000 C CNN
+F 1 "4.7k" V 7934 5550 50  0000 C CNN
+F 2 "Resistors_SMD:R_0603" V 7980 5550 50  0001 C CNN
+F 3 "" H 8050 5550 50  0001 C CNN
+F 4 "Yageo" H 8050 5550 50  0001 C CNN "MFN"
+F 5 "RC0603FR-074K7L" H 8050 5550 50  0001 C CNN "MFP"
+	1    8050 5550
+	0    1    1    0
+$EndComp
+Wire Wire Line
+	8350 5550 8200 5550
+Wire Wire Line
+	7900 5550 6700 5550
+Wire Wire Line
+	6700 3100 6700 5550
+Text Notes 9250 5650 0    50   ~ 0
+We are using a transistor\nso that we can isolate the\npin using a 4.7k resistor
 $EndSCHEMATC

Commit message: Updated to Kicad v5.0
Parts:
- removed J7: AVR-ISP-6, Pin_Headers:Pin_Header_Straight_2x03_Pitch2.54mm, symbol atmel:AVR-ISP-6
- removed U4: ATTINY13, Housings_SOIC:SOIC-8_3.9x4.9mm_Pitch1.27mm, symbol atmel:ATTINY13-20SSU
- added J7: AVR-ISP-6, Connector_PinHeader_2.54mm:PinHeader_2x03_P2.54mm_Vertical, symbol Connector:AVR-ISP-6
- added U4: ATtiny13-20SSU, Package_SO:SOIC-8_3.9x4.9mm_P1.27mm, symbol MCU_Microchip_ATtiny:ATtiny13-20SSU
- C10, C11, C12: symbol device:C -> Device:C
- J6: symbol conn:Conn_01x02 -> Connector_Generic:Conn_01x02
- Q3: symbol transistors:MMBT3904 -> Transistor_BJT:MMBT3904
- R13, R14, R15, R16, R17, R18: symbol device:R -> Device:R
- SW2: symbol switches:SW_SPDT -> Switch:SW_SPDT
Connections:
- wire segments 58 -> 55
Other:
- moved on the sheet: C10, R16
Changed lines of the file:
@@
 Text HLabel 5250 4550 0    60   Input ~ 0
 ADC_in
-Text HLabel 3350 3000 0    60   UnSpc ~ 0
+Text HLabel 5150 1900 1    60   UnSpc ~ 0
 Vdd
 Text HLabel 7650 3700 2    60   Output ~ 0
 ~enable_heater
 $Comp
-L device:R R13
+L Device:R R13
 U 1 1 59D0B837
 P 5550 4550
@@
 $EndComp
 $Comp
-L device:C C11
+L Device:C C11
 U 1 1 59D0B89F
 P 5850 4800
@@
 $EndComp
 $Comp
-L atmel:ATTINY13-20SSU U4
-U 1 1 59D0BE2F
-P 5300 3250
-F 0 "U4" H 5300 3767 50  0000 C CNN
-F 1 "ATTINY13" H 5300 3676 50  0000 C CNN
-F 2 "Housings_SOIC:SOIC-8_3.9x4.9mm_Pitch1.27mm" H 5900 3250 50  0001 C CIN
-F 3 "" H 4500 3600 50  0001 C CNN
-F 4 "Microchip Technology" H 5300 3250 60  0001 C CNN "MFN"
-F 5 "ATTINY13A-SS7" H 5300 3250 60  0001 C CNN "MFP"
-	1    5300 3250
-	-1   0    0    -1
-$EndComp
-$Comp
 L power:GND #PWR025
 U 1 1 59D0C06D
-P 4100 3600
-F 0 "#PWR025" H 4100 3350 50  0001 C CNN
-F 1 "GND" H 4105 3427 50  0000 C CNN
-F 2 "" H 4100 3600 50  0001 C CNN
-F 3 "" H 4100 3600 50  0001 C CNN
-	1    4100 3600
+P 5150 4000
+F 0 "#PWR025" H 5150 3750 50  0001 C CNN
+F 1 "GND" H 5155 3827 50  0000 C CNN
+F 2 "" H 5150 4000 50  0001 C CNN
+F 3 "" H 5150 4000 50  0001 C CNN
+	1    5150 4000
 	1    0    0    -1
 $EndComp
@@
 L power:GND #PWR030
 U 1 1 59D0C22E
-P 8000 2750
-F 0 "#PWR030" H 8000 2500 50  0001 C CNN
-F 1 "GND" H 8005 2577 50  0000 C CNN
-F 2 "" H 8000 2750 50  0001 C CNN
-F 3 "" H 8000 2750 50  0001 C CNN
-	1    8000 2750
-	1    0    0    -1
-$EndComp
-Text HLabel 9350 2500 2    60   UnSpc ~ 0
+P 8150 3200
+F 0 "#PWR030" H 8150 2950 50  0001 C CNN
+F 1 "GND" H 8155 3027 50  0000 C CNN
+F 2 "" H 8150 3200 50  0001 C CNN
+F 3 "" H 8150 3200 50  0001 C CNN
+	1    8150 3200
+	-1   0    0    -1
+$EndComp
+Text HLabel 8150 2000 1    60   UnSpc ~ 0
 Vdd
 $Comp
-L device:R R16
+L Device:R R16
 U 1 1 59D0C448
-P 8600 2900
-F 0 "R16" H 8670 2946 50  0000 L CNN
-F 1 "10k" H 8670 2855 50  0000 L CNN
-F 2 "Resistors_SMD:R_0603" V 8530 2900 50  0001 C CNN
-F 3 "" H 8600 2900 50  0001 C CNN
-F 4 "Yageo" H 8600 2900 60  0001 C CNN "MFN"
-F 5 "RC0603JR-0710KL" H 8600 2900 60  0001 C CNN "MFP"
-	1    8600 2900
-	1    0    0    -1
-$EndComp
-$Comp
-L device:C C10
+P 9000 2900
+F 0 "R16" H 9070 2946 50  0000 L CNN
+F 1 "10k" H 9070 2855 50  0000 L CNN
+F 2 "Resistors_SMD:R_0603" V 8930 2900 50  0001 C CNN
+F 3 "" H 9000 2900 50  0001 C CNN
+F 4 "Yageo" H 9000 2900 60  0001 C CNN "MFN"
+F 5 "RC0603JR-0710KL" H 9000 2900 60  0001 C CNN "MFP"
+	1    9000 2900
+	1    0    0    -1
+$EndComp
+$Comp
+L Device:C C10
 U 1 1 59D0C55B
-P 3700 3400
-F 0 "C10" H 3815 3446 50  0000 L CNN
-F 1 "100n" H 3815 3355 50  0000 L CNN
-F 2 "Capacitors_SMD:C_0603" H 3738 3250 50  0001 C CNN
-F 3 "" H 3700 3400 50  0001 C CNN
-F 4 "Murata" H 3700 3400 60  0001 C CNN "MFN"
-F 5 "GRM188R71H104KA93D" H 3700 3400 60  0001 C CNN "MFP"
-	1    3700 3400
+P 4700 2250
+F 0 "C10" H 4815 2296 50  0000 L CNN
+F 1 "100n" H 4815 2205 50  0000 L CNN
+F 2 "Capacitors_SMD:C_0603" H 4738 2100 50  0001 C CNN
+F 3 "" H 4700 2250 50  0001 C CNN
+F 4 "Murata" H 4700 2250 60  0001 C CNN "MFN"
+F 5 "GRM188R71H104KA93D" H 4700 2250 60  0001 C CNN "MFP"
+	1    4700 2250
 	1    0    0    -1
 $EndComp
@@
 L power:GND #PWR024
 U 1 1 59D0C561
-P 3700 3650
-F 0 "#PWR024" H 3700 3400 50  0001 C CNN
-F 1 "GND" H 3705 3477 50  0000 C CNN
-F 2 "" H 3700 3650 50  0001 C CNN
-F 3 "" H 3700 3650 50  0001 C CNN
-	1    3700 3650
+P 4700 2500
+F 0 "#PWR024" H 4700 2250 50  0001 C CNN
+F 1 "GND" H 4705 2327 50  0000 C CNN
+F 2 "" H 4700 2500 50  0001 C CNN
+F 3 "" H 4700 2500 50  0001 C CNN
+	1    4700 2500
 	1    0    0    -1
 $EndComp
@@
 ~kill_power
 $Comp
-L device:R R15
+L Device:R R15
 U 1 1 59D0EA56
 P 8650 4850
@@
 $EndComp
 $Comp
-L switches:SW_SPDT SW2
+L Switch:SW_SPDT SW2
 U 1 1 59D116BA
 P 6700 1900
@@
 $EndComp
 $Comp
-L conn:Conn_01x02 J6
+L Connector_Generic:Conn_01x02 J6
 U 1 1 59D151F1
 P 8900 5150
@@
 $EndComp
 $Comp
-L device:C C12
+L Device:C C12
 U 1 1 59D1A6E6
 P 6050 2100
@@
 	5850 4950 5850 5050
 Wire Wire Line
-	3350 3000 3700 3000
-Wire Wire Line
-	4300 3500 4100 3500
-Wire Wire Line
-	4100 3500 4100 3600
-Wire Wire Line
-	7150 2500 7500 2500
-Wire Wire Line
-	6300 3100 6700 3100
-Wire Wire Line
-	7250 2600 7500 2600
-Wire Wire Line
-	7250 2600 7250 3200
-Wire Wire Line
-	7250 3200 6400 3200
-Wire Wire Line
-	7350 2700 7500 2700
-Wire Wire Line
-	7350 2700 7350 3500
-Wire Wire Line
-	6300 3500 7350 3500
-Wire Wire Line
-	6300 3000 6850 3000
-Wire Wire Line
-	8300 3000 8300 2600
-Wire Wire Line
-	8300 2600 7750 2600
-Wire Wire Line
-	7750 2700 8000 2700
-Wire Wire Line
-	8000 2700 8000 2750
-Wire Wire Line
-	8600 2500 8600 2750
-Connection ~ 8600 2500
-Wire Wire Line
-	8600 3500 8600 3050
-Connection ~ 7350 3500
-Wire Wire Line
-	3700 3550 3700 3650
-Wire Wire Line
-	3700 3250 3700 3000
-Connection ~ 3700 3000
-Wire Wire Line
-	7150 3700 7650 3700
-Wire Wire Line
-	6850 4050 7650 4050
+	5150 3900 5150 4000
+Wire Wire Line
+	6850 2500 7650 2500
+Wire Wire Line
+	5750 3100 6700 3100
+Wire Wire Line
+	7050 2700 7650 2700
+Wire Wire Line
+	7050 2700 7050 3200
+Wire Wire Line
+	7050 3200 6400 3200
+Wire Wire Line
+	7150 2800 7650 2800
+Wire Wire Line
+	7150 2800 7150 3500
+Wire Wire Line
+	5750 3500 7150 3500
+Wire Wire Line
+	5750 3000 6950 3000
+Wire Wire Line
+	9000 2500 9000 2750
+Wire Wire Line
+	9000 3500 9000 3050
+Connection ~ 7150 3500
+Wire Wire Line
+	4700 2400 4700 2500
+Wire Wire Line
+	7050 3700 7650 3700
+Wire Wire Line
+	6950 4050 7650 4050
 Wire Wire Line
 	6550 4550 6550 3400
 Wire Wire Line
-	6550 3400 6300 3400
+	6550 3400 5750 3400
 Connection ~ 5850 4550
 Wire Wire Line
@@
 	7050 1800 7050 1900
 Wire Wire Line
-	6850 4050 6850 3000
-Connection ~ 6850 3000
+	6950 4050 6950 3000
 Wire Wire Line
 	8650 5150 8700 5150
@@
 Wire Wire Line
 	6050 2300 6050 2250
-Wire Wire Line
-	7750 2500 8600 2500
 Text Label 6500 3500 0    60   ~ 0
 RST
@@
 SCK
 Wire Wire Line
-	7150 3100 7150 2500
-Wire Wire Line
-	7150 3300 7150 3700
-Wire Wire Line
-	6300 3300 7150 3300
-$Comp
-L device:R R14
+	6850 3100 6850 2500
+Wire Wire Line
+	7050 3300 7050 3700
+Wire Wire Line
+	5750 3300 7050 3300
+$Comp
+L Device:R R14
 U 1 1 5A46E3DE
 P 6400 2500
@@
 	6400 2650 6400 3200
 Connection ~ 6400 3200
-$Comp
-L atmel:AVR-ISP-6 J7
-U 1 1 5A46F178
-P 7650 2600
-F 0 "J7" H 7637 2965 50  0000 C CNN
-F 1 "AVR-ISP-6" H 7637 2874 50  0000 C CNN
-F 2 "Pin_Headers:Pin_Header_Straight_2x03_Pitch2.54mm" V 7130 2640 50  0001 C CNN
-F 3 "" H 7625 2600 50  0001 C CNN
-	1    7650 2600
-	1    0    0    -1
-$EndComp
-Wire Wire Line
-	8600 2500 9350 2500
-Wire Wire Line
-	7350 3500 8600 3500
-Wire Wire Line
-	3700 3000 4300 3000
+Wire Wire Line
+	7150 3500 9000 3500
 Wire Wire Line
 	5850 4550 6550 4550
 Wire Wire Line
-	6700 3100 7150 3100
-Wire Wire Line
-	6850 3000 8300 3000
+	6700 3100 6850 3100
 Wire Wire Line
 	6400 1900 6500 1900
 Wire Wire Line
-	6400 3200 6300 3200
-$Comp
-L device:R R17
+	6400 3200 5750 3200
+$Comp
+L Device:R R17
 U 1 1 5AAF2F34
 P 7800 4050
@@
 	8650 4500 8650 4700
 $Comp
-L transistors:MMBT3904 Q3
+L Transistor_BJT:MMBT3904 Q3
 U 1 1 5AAF71EA
 P 8550 5550
@@
 	8650 5250 8650 5350
 $Comp
-L device:R R18
+L Device:R R18
 U 1 1 5AAF9A93
 P 8050 5550
@@
 Text Notes 9250 5650 0    50   ~ 0
 We are using a transistor\nso that we can isolate the\npin using a 4.7k resistor
+Wire Wire Line
+	5150 1900 5150 2050
+Wire Wire Line
+	4700 2100 4700 2050
+Wire Wire Line
+	4700 2050 5150 2050
+Connection ~ 5150 2050
+Wire Wire Line
+	5150 2050 5150 2700
+$Comp
+L MCU_Microchip_ATtiny:ATtiny13-20SSU U4
+U 1 1 5B07BB44
+P 5150 3300
+F 0 "U4" H 4620 3346 50  0000 R CNN
+F 1 "ATtiny13-20SSU" H 4620 3255 50  0000 R CNN
+F 2 "Package_SO:SOIC-8_3.9x4.9mm_P1.27mm" H 5150 3300 50  0001 C CIN
+F 3 "http://ww1.microchip.com/downloads/en/DeviceDoc/doc2535.pdf" H 5150 3300 50  0001 C CNN
+	1    5150 3300
+	1    0    0    -1
+$EndComp
+$Comp
+L Connector:AVR-ISP-6 J7
+U 1 1 5B089944
+P 8050 2700
+F 0 "J7" H 7770 2796 50  0000 R CNN
+F 1 "AVR-ISP-6" H 7770 2705 50  0000 R CNN
+F 2 "Connector_PinHeader_2.54mm:PinHeader_2x03_P2.54mm_Vertical" V 7800 2750 50  0001 C CNN
+F 3 " ~" H 6775 2150 50  0001 C CNN
+	1    8050 2700
+	-1   0    0    -1
+$EndComp
+Wire Wire Line
+	8150 3100 8150 3200
+Wire Wire Line
+	6950 3000 6950 2600
+Wire Wire Line
+	6950 2600 7650 2600
+Connection ~ 6950 3000
+Wire Wire Line
+	8150 2000 8150 2200
+Text HLabel 9000 2500 1    60   UnSpc ~ 0
+Vdd
 $EndSCHEMATC
