File: boost_converter.sch (KiCad schematic (older format))
At the start: 21 parts, among them J4 GS2, J5 GS2, J8 Conn_01x01, SW1 SW_Push, U2 LTC2955-1(DFN), U3 LTC3536

Commit message: Updated to Kicad v5.0
Parts:
- removed J4, J5: GS2, Custom_footprints:jumper_solder_small, symbol conn:GS2
- removed J8: Conn_01x01, Measurement_Points:Measurement_Point_Round-SMD-Pad_Small, symbol conn:Conn_01x01
- added JP1, JP2: SolderJumper_2_Open, Jumper:SolderJumper-2_P1.3mm_Open_RoundedPad1.0x1.5mm, symbol Jumper:SolderJumper_2_Open
- added TP1: Test_Point, TestPoint:TestPoint_Pad_D1.5mm, symbol Connector:Test_Point
- C3, C4, C5, C6, C7, C8, C9: symbol device:C -> Device:C
- L1: symbol device:L -> Device:L
- R10, R11, R12, R6, R7, R8, R9: symbol device:R -> Device:R
- SW1: symbol switches:SW_Push -> Switch:SW_Push
Other:
- note added: "Optional:\nClose JP1 for debugging\nto always enable the DC/DC\nconverter"
- note added: "Optional:\nClose JP2 for debugging\nto keep the DC/DC converter enabled"
- note removed: "Optional:\nClose J4 for debugging\nto always enable the DC/DC\nconverter"
- note removed: "Optional:\nClose J5 for debugging\nto keep the DC/DC converter enabled"
Changed lines of the file:
@@
 Vsup
 $Comp
-L device:C C3
+L Device:C C3
 U 1 1 59D07029
 P 3300 4300
@@
 $EndComp
 $Comp
-L switches:SW_Push SW1
+L Switch:SW_Push SW1
 U 1 1 59D0729E
 P 4100 4750
@@
 $EndComp
 $Comp
-L device:C C5
+L Device:C C5
 U 1 1 59D073A5
 P 4700 5050
@@
 $EndComp
 $Comp
-L device:R R6
+L Device:R R6
 U 1 1 59D07A41
 P 2300 3800
@@
 $EndComp
 $Comp
-L device:R R8
+L Device:R R8
 U 1 1 59D08F18
 P 5100 2300
@@
 V+5
 $Comp
-L device:R R12
+L Device:R R12
 U 1 1 59D096F1
 P 7750 1950
@@
 $EndComp
 $Comp
-L device:R R11
+L Device:R R11
 U 1 1 59D09D45
 P 7350 1950
@@
 $EndComp
 $Comp
-L device:C C7
+L Device:C C7
 U 1 1 59D09F1D
 P 7350 2300
@@
 $EndComp
 $Comp
-L device:R R10
+L Device:R R10
 U 1 1 59D0A192
 P 6850 2750
@@
 $EndComp
 $Comp
-L device:C C6
+L Device:C C6
 U 1 1 59D0A27C
 P 6850 2350
@@
 $EndComp
 $Comp
-L device:L L1
+L Device:L L1
 U 1 1 59D0A787
 P 5750 1150
@@
 	5150 1150 5150 1650
 $Comp
-L device:C C4
+L Device:C C4
 U 1 1 59D0AC39
 P 3550 2000
@@
 	3550 1850 3550 1750
 $Comp
-L device:C C8
+L Device:C C8
 U 1 1 59D0AF6C
 P 8300 2000
@@
 	4050 2600 4050 2700
 $Comp
-L device:R R7
+L Device:R R7
 U 1 1 5A46F9EB
 P 4050 2450
@@
 	9450 1750 9550 1750
 Wire Wire Line
-	5950 4050 5950 4150
+	5950 3950 5950 4150
 Connection ~ 5950 4150
 Wire Wire Line
@@
 	6850 2500 6850 2550
 $Comp
-L device:R R9
+L Device:R R9
 U 1 1 5AAEC85B
 P 6550 2050
@@
 	7750 1750 8300 1750
 $Comp
-L device:C C9
+L Device:C C9
 U 1 1 5AB03DE0
 P 8750 2000
@@
 Wire Wire Line
 	4400 1950 4850 1950
-Wire Wire Line
-	4050 2250 4050 2200
 Connection ~ 4050 2250
 Wire Notes Line
@@
 	3850 2950 3850 1600
 Text Notes 3800 1500 0    50   ~ 0
-Optional:\nClose J4 for debugging\nto always enable the DC/DC\nconverter
-$Comp
-L conn:GS2 J4
-U 1 1 5AB17422
-P 4050 2000
-F 0 "J4" H 4118 2046 50  0000 L CNN
-F 1 "GS2" H 4118 1955 50  0000 L CNN
-F 2 "Custom_footprints:jumper_solder_small" V 4124 2000 50  0001 C CNN
-F 3 "" H 4050 2000 50  0001 C CNN
-	1    4050 2000
-	1    0    0    -1
-$EndComp
-$Comp
-L conn:GS2 J5
-U 1 1 5AB20F4D
-P 5950 3850
-F 0 "J5" H 6018 3896 50  0000 L CNN
-F 1 "GS2" H 6018 3805 50  0000 L CNN
-F 2 "Custom_footprints:jumper_solder_small" V 6024 3850 50  0001 C CNN
-F 3 "" H 5950 3850 50  0001 C CNN
-	1    5950 3850
-	1    0    0    -1
-$EndComp
-Text Notes 6350 3950 0    50   ~ 0
-Optional:\nClose J5 for debugging\nto keep the DC/DC converter enabled
-$Comp
-L conn:Conn_01x01 J8
-U 1 1 5AAF1D34
-P 9100 1400
-F 0 "J8" V 9066 1312 50  0000 R CNN
-F 1 "Conn_01x01" V 8975 1312 50  0000 R CNN
-F 2 "Measurement_Points:Measurement_Point_Round-SMD-Pad_Small" H 9100 1400 50  0001 C CNN
-F 3 "~" H 9100 1400 50  0001 C CNN
-	1    9100 1400
-	0    -1   -1   0
-$EndComp
+Optional:\nClose JP1 for debugging\nto always enable the DC/DC\nconverter
+Text Notes 6250 3750 0    50   ~ 0
+Optional:\nClose JP2 for debugging\nto keep the DC/DC converter enabled
 Wire Wire Line
 	9100 1600 9100 1750
@@
 Wire Wire Line
 	9100 1750 9450 1750
+Wire Wire Line
+	4050 2100 4050 2250
+$Comp
+L Jumper:SolderJumper_2_Open JP1
+U 1 1 5B07240D
+P 4050 1950
+F 0 "JP1" V 4004 2018 50  0000 L CNN
+F 1 "SolderJumper_2_Open" V 4095 2018 50  0000 L CNN
+F 2 "Jumper:SolderJumper-2_P1.3mm_Open_RoundedPad1.0x1.5mm" H 4050 1950 50  0001 C CNN
+F 3 "~" H 4050 1950 50  0001 C CNN
+	1    4050 1950
+	0    1    1    0
+$EndComp
+$Comp
+L Jumper:SolderJumper_2_Open JP2
+U 1 1 5B0731E9
+P 5950 3800
+F 0 "JP2" V 5904 3868 50  0000 L CNN
+F 1 "SolderJumper_2_Open" V 5995 3868 50  0000 L CNN
+F 2 "Jumper:SolderJumper-2_P1.3mm_Open_RoundedPad1.0x1.5mm" H 5950 3800 50  0001 C CNN
+F 3 "~" H 5950 3800 50  0001 C CNN
+	1    5950 3800
+	0    1    1    0
+$EndComp
+$Comp
+L Connector:Test_Point TP1
+U 1 1 5B075D2B
+P 9100 1600
+F 0 "TP1" H 9158 1720 50  0000 L CNN
+F 1 "Test_Point" H 9158 1629 50  0000 L CNN
+F 2 "TestPoint:TestPoint_Pad_D1.5mm" H 9300 1600 50  0001 C CNN
+F 3 "~" H 9300 1600 50  0001 C CNN
+	1    9100 1600
+	1    0    0    -1
+$EndComp
 $EndSCHEMATC

Commit message: Added power on state LED Updated to KiCAD 5.0
Parts:
- added D3: LED, LED_SMD:LED_0805_2012Metric, symbol Device:LED
- added R19: 1k, Resistor_SMD:R_0603_1608Metric, symbol Device:R
- C3, C5, C6, C7: footprint Capacitors_SMD:C_0603 -> Capacitor_SMD:C_0603_1608Metric
- C4, C8, C9: footprint Capacitors_SMD:C_0805 -> Capacitor_SMD:C_0805_2012Metric
- R10, R11, R12, R6, R7, R8, R9: footprint Resistors_SMD:R_0603 -> Resistor_SMD:R_0603_1608Metric
- U2: footprint Housings_DFN_QFN:DFN-10-1EP_2x3mm_Pitch0.5mm -> Package_DFN_QFN:DFN-10-1EP_2x3mm_P0.5mm_EP0.64x2.4mm
- U3: footprint Housings_DFN_QFN:DFN-10-1EP_3x3mm_Pitch0.5mm -> Package_DFN_QFN:DFN-10-1EP_3x3mm_P0.5mm_EP1.55x2.48mm
Connections:
- wire segments 82 -> 88
- no-connect marks 0 -> 2
Other:
- note added: "The LTC2955 requires only 1.2 µA \nof current so the 1k resistor is OK\nand it allows reverse input."
Changed lines of the file:
@@
 F 0 "U2" H 5000 5050 60  0000 C CNN
 F 1 "LTC2955-1(DFN)" H 5300 4950 60  0000 C CNN
-F 2 "Housings_DFN_QFN:DFN-10-1EP_2x3mm_Pitch0.5mm" H 6200 5050 60  0001 C CNN
+F 2 "Package_DFN_QFN:DFN-10-1EP_2x3mm_P0.5mm_EP0.64x2.4mm" H 6200 5050 60  0001 C CNN
 F 3 "" H 4900 4350 60  0000 C CNN
 F 4 "Linear Technology" H 5200 4250 60  0001 C CNN "MFN"
@@
 F 0 "C3" H 3415 4346 50  0000 L CNN
 F 1 "10n" H 3415 4255 50  0000 L CNN
-F 2 "Capacitors_SMD:C_0603" H 3338 4150 50  0001 C CNN
+F 2 "Capacitor_SMD:C_0603_1608Metric" H 3338 4150 50  0001 C CNN
 F 3 "" H 3300 4300 50  0001 C CNN
 F 4 "Murata" H 3300 4300 60  0001 C CNN "MFN"
@@
 F 0 "C5" H 4815 5096 50  0000 L CNN
 F 1 "100n" H 4815 5005 50  0000 L CNN
-F 2 "Capacitors_SMD:C_0603" H 4738 4900 50  0001 C CNN
+F 2 "Capacitor_SMD:C_0603_1608Metric" H 4738 4900 50  0001 C CNN
 F 3 "" H 4700 5050 50  0001 C CNN
 F 4 "Murata" H 4700 5050 60  0001 C CNN "MFN"
@@
 F 0 "R6" H 2370 3846 50  0000 L CNN
 F 1 "1k" H 2370 3755 50  0000 L CNN
-F 2 "Resistors_SMD:R_0603" V 2230 3800 50  0001 C CNN
+F 2 "Resistor_SMD:R_0603_1608Metric" V 2230 3800 50  0001 C CNN
 F 3 "" H 2300 3800 50  0001 C CNN
 F 4 "Yageo" H 2300 3800 60  0001 C CNN "MFN"
@@
 F 0 "R8" H 5170 2346 50  0000 L CNN
 F 1 "332k" H 5170 2255 50  0000 L CNN
-F 2 "Resistors_SMD:R_0603" V 5030 2300 50  0001 C CNN
+F 2 "Resistor_SMD:R_0603_1608Metric" V 5030 2300 50  0001 C CNN
 F 3 "" H 5100 2300 50  0001 C CNN
 F 4 "Yageo" H 5100 2300 60  0001 C CNN "MFN"
@@
 	1    0    0    -1
 $EndComp
-Text HLabel 9550 1750 2    60   UnSpc ~ 0
+Text HLabel 10800 1750 2    60   UnSpc ~ 0
 V+5
 $Comp
@@
 F 0 "R12" H 7820 1996 50  0000 L CNN
 F 1 "1.1M" H 7820 1905 50  0000 L CNN
-F 2 "Resistors_SMD:R_0603" V 7680 1950 50  0001 C CNN
+F 2 "Resistor_SMD:R_0603_1608Metric" V 7680 1950 50  0001 C CNN
 F 3 "" H 7750 1950 50  0001 C CNN
 F 4 "Yageo" H 7750 1950 60  0001 C CNN "MFN"
@@
 F 0 "R11" H 7420 1996 50  0000 L CNN
 F 1 "22.6k" H 7420 1905 50  0000 L CNN
-F 2 "Resistors_SMD:R_0603" V 7280 1950 50  0001 C CNN
+F 2 "Resistor_SMD:R_0603_1608Metric" V 7280 1950 50  0001 C CNN
 F 3 "" H 7350 1950 50  0001 C CNN
 F 4 "Susumu" H 7350 1950 60  0001 C CNN "MFN"
@@
 F 0 "C7" H 7465 2346 50  0000 L CNN
 F 1 "18p" H 7465 2255 50  0000 L CNN
-F 2 "Capacitors_SMD:C_0603" H 7388 2150 50  0001 C CNN
+F 2 "Capacitor_SMD:C_0603_1608Metric" H 7388 2150 50  0001 C CNN
 F 3 "" H 7350 2300 50  0001 C CNN
 F 4 "Kemet" H 7350 2300 60  0001 C CNN "MFN"
@@
 F 0 "R10" H 6920 2796 50  0000 L CNN
 F 1 "150k" H 6920 2705 50  0000 L CNN
-F 2 "Resistors_SMD:R_0603" V 6780 2750 50  0001 C CNN
+F 2 "Resistor_SMD:R_0603_1608Metric" V 6780 2750 50  0001 C CNN
 F 3 "" H 6850 2750 50  0001 C CNN
 F 4 "Susumu" H 6850 2750 60  0001 C CNN "MFN"
@@
 F 0 "C6" H 6965 2396 50  0000 L CNN
 F 1 "200p" H 6965 2305 50  0000 L CNN
-F 2 "Capacitors_SMD:C_0603" H 6888 2200 50  0001 C CNN
+F 2 "Capacitor_SMD:C_0603_1608Metric" H 6888 2200 50  0001 C CNN
 F 3 "" H 6850 2350 50  0001 C CNN
 F 4 "Kemet" H 6850 2350 60  0001 C CNN "MFN"
@@
 F 0 "C4" H 3665 2046 50  0000 L CNN
 F 1 "47u" H 3665 1955 50  0000 L CNN
-F 2 "Capacitors_SMD:C_0805" H 3588 1850 50  0001 C CNN
+F 2 "Capacitor_SMD:C_0805_2012Metric" H 3588 1850 50  0001 C CNN
 F 3 "" H 3550 2000 50  0001 C CNN
 F 4 "Murata" H 3550 2000 60  0001 C CNN "MFN"
@@
 F 0 "C8" H 8415 2046 50  0000 L CNN
 F 1 "47u" H 8415 1955 50  0000 L CNN
-F 2 "Capacitors_SMD:C_0805" H 8338 1850 50  0001 C CNN
+F 2 "Capacitor_SMD:C_0805_2012Metric" H 8338 1850 50  0001 C CNN
 F 3 "" H 8300 2000 50  0001 C CNN
 F 4 "Murata" H 8300 2000 60  0001 C CNN "MFN"
@@
 F 0 "R7" H 4120 2496 50  0000 L CNN
 F 1 "100k" H 4120 2405 50  0000 L CNN
-F 2 "Resistors_SMD:R_0603" H 4120 2359 50  0001 L CNN
+F 2 "Resistor_SMD:R_0603_1608Metric" H 4120 2359 50  0001 L CNN
 F 3 "" H 4050 2450 50  0000 C CNN
 F 4 "Yageo" H 4050 2450 60  0001 C CNN "MFN"
@@
 	2300 2650 2300 3650
 Wire Wire Line
-	3300 4050 4300 4050
+	3300 4050 3600 4050
 Wire Wire Line
 	5150 1650 5200 1650
@@
 Connection ~ 9450 1750
 Wire Wire Line
-	9450 1750 9550 1750
+	9450 1750 9850 1750
 Wire Wire Line
 	5950 3950 5950 4150
@@
 F 0 "U3" H 5750 2637 60  0000 C CNN
 F 1 "LTC3536" H 5750 2531 60  0000 C CNN
-F 2 "Housings_DFN_QFN:DFN-10-1EP_3x3mm_Pitch0.5mm" H 7100 2650 60  0001 C CNN
+F 2 "Package_DFN_QFN:DFN-10-1EP_3x3mm_P0.5mm_EP1.55x2.48mm" H 7100 2650 60  0001 C CNN
 F 3 "https://cds.linear.com/docs/en/datasheet/3458fa.pdf" H 5750 2531 60  0001 C CNN
 F 4 "Linear Technology" H 6750 1350 60  0001 C CNN "MFN"
@@
 F 0 "R9" V 6343 2050 50  0000 C CNN
 F 1 "33k" V 6434 2050 50  0000 C CNN
-F 2 "Resistors_SMD:R_0603" V 6480 2050 50  0001 C CNN
+F 2 "Resistor_SMD:R_0603_1608Metric" V 6480 2050 50  0001 C CNN
 F 3 "" H 6550 2050 50  0001 C CNN
 F 4 "Susumu" H 6550 2050 50  0001 C CNN "MFN"
@@
 F 0 "C9" H 8865 2046 50  0000 L CNN
 F 1 "47u" H 8865 1955 50  0000 L CNN
-F 2 "Capacitors_SMD:C_0805" H 8788 1850 50  0001 C CNN
+F 2 "Capacitor_SMD:C_0805_2012Metric" H 8788 1850 50  0001 C CNN
 F 3 "" H 8750 2000 50  0001 C CNN
 F 4 "Murata" H 8750 2000 60  0001 C CNN "MFN"
@@
 	1    0    0    -1
 $EndComp
+$Comp
+L Device:R R19
+U 1 1 5B1CB81C
+P 9850 2000
+F 0 "R19" H 9920 2046 50  0000 L CNN
+F 1 "1k" H 9920 1955 50  0000 L CNN
+F 2 "Resistor_SMD:R_0603_1608Metric" V 9780 2000 50  0001 C CNN
+F 3 "~" H 9850 2000 50  0001 C CNN
+	1    9850 2000
+	1    0    0    -1
+$EndComp
+$Comp
+L Device:LED D3
+U 1 1 5B1CBA70
+P 9850 2400
+F 0 "D3" V 9888 2283 50  0000 R CNN
+F 1 "LED" V 9797 2283 50  0000 R CNN
+F 2 "LED_SMD:LED_0805_2012Metric" H 9850 2400 50  0001 C CNN
+F 3 "~" H 9850 2400 50  0001 C CNN
+	1    9850 2400
+	0    -1   -1   0
+$EndComp
+$Comp
+L power:GND #PWR0101
+U 1 1 5B1CBB32
+P 9850 2650
+F 0 "#PWR0101" H 9850 2400 50  0001 C CNN
+F 1 "GND" H 9855 2477 50  0000 C CNN
+F 2 "" H 9850 2650 50  0001 C CNN
+F 3 "" H 9850 2650 50  0001 C CNN
+	1    9850 2650
+	1    0    0    -1
+$EndComp
+Wire Wire Line
+	9850 2650 9850 2550
+Wire Wire Line
+	9850 2250 9850 2150
+Wire Wire Line
+	9850 1850 9850 1750
+Connection ~ 9850 1750
+Wire Wire Line
+	9850 1750 10800 1750
+NoConn ~ 5400 4050
+NoConn ~ 5400 4250
+$Comp
+L power:PWR_FLAG #FLG0101
+U 1 1 5B1DE48F
+P 3600 3900
+F 0 "#FLG0101" H 3600 3975 50  0001 C CNN
+F 1 "PWR_FLAG" H 3600 4074 50  0000 C CNN
+F 2 "" H 3600 3900 50  0001 C CNN
+F 3 "~" H 3600 3900 50  0001 C CNN
+	1    3600 3900
+	1    0    0    -1
+$EndComp
+Wire Wire Line
+	3600 3900 3600 4050
+Connection ~ 3600 4050
+Wire Wire Line
+	3600 4050 4300 4050
+Text Notes 3000 3650 0    50   ~ 0
+The LTC2955 requires only 1.2 µA \nof current so the 1k resistor is OK\nand it allows reverse input.
 $EndSCHEMATC

Commit message: Added part numbers Updated BOM
Parts:
- D3: MFN (none) -> Kingbright; MFP (none) -> APT2012VBC/D
- R19: MFN (none) -> Yageo; MFP (none) -> RC0603FR-071KL
Changed lines of the file:
@@
 F 2 "Resistor_SMD:R_0603_1608Metric" V 9780 2000 50  0001 C CNN
 F 3 "~" H 9850 2000 50  0001 C CNN
+F 4 "Yageo" H 9850 2000 50  0001 C CNN "MFN"
+F 5 "RC0603FR-071KL" H 9850 2000 50  0001 C CNN "MFP"
 	1    9850 2000
 	1    0    0    -1
@@
 F 2 "LED_SMD:LED_0805_2012Metric" H 9850 2400 50  0001 C CNN
 F 3 "~" H 9850 2400 50  0001 C CNN
+F 4 "Kingbright" H 9850 2400 50  0001 C CNN "MFN"
+F 5 "APT2012VBC/D" H 9850 2400 50  0001 C CNN "MFP"
 	1    9850 2400
 	0    -1   -1   0

Commit message: Changed description of the blue LED
Parts:
- D3: value LED -> Blue LED
Changed lines of the file:
@@
 P 9850 2400
 F 0 "D3" V 9888 2283 50  0000 R CNN
-F 1 "LED" V 9797 2283 50  0000 R CNN
+F 1 "Blue LED" V 9797 2283 50  0000 R CNN
 F 2 "LED_SMD:LED_0805_2012Metric" H 9850 2400 50  0001 C CNN
 F 3 "~" H 9850 2400 50  0001 C CNN
